File: Hardware/PCB/IOs stage.kicad_sch (KiCad schematic)
At the start: 30 parts, among them IC11 LP5951MFX-3.3/NOPB, IC12 SI8621BC, IC13 SI8621BC, IC14 SI8621BC, IC15 SI8621BC, IC16 SI8621BC, IC17 SI8621BC

Commit message: commit para revisão do Filipe
Parts:
- removed CLKIN0, CLKOUT0, CLKOUT1, CLKOUT2, CLKOUT3, CLKOUT4, CLKOUT5: 35RASMT2BHNTRX, harp_timestamp_generator_Gen3:35RASMT2BHNTRX, symbol harp_timestamp_generator_Gen3:35RASMT2BHNTRX
- added CLKIN0, CLKOUT0, CLKOUT1, CLKOUT2, CLKOUT3, CLKOUT4, CLKOUT5: 35RASMT2BHNTRX, harp_timestamp_generator_Gen3:35RASMT2BHNTRX, symbol Connector_Audio:AudioJack2_Ground
Connections:
- net CLOCK_IN: now also CLKIN0.2
- net GND: now also CLKIN0.1
- net at R2.2, R3.1: now also CLKIN0.3
- net at C26.1, IC12.6 (B2_IN), IC12.8 (BVDD): now also CLKOUT0.3
- net at C26.2, IC12.5 (BGND): now also CLKOUT0.1
- net at C21.2, IC17.5 (BGND): now also CLKOUT5.1
- net at IC17.7 (B1_OUT): now also CLKOUT5.2
- net at C21.1, IC17.6 (B2_IN), IC17.8 (BVDD): now also CLKOUT5.3
- net at IC12.7 (B1_OUT): now also CLKOUT0.2
- net at C17.1, IC15.6 (B2_IN), IC15.8 (BVDD): now also CLKOUT3.3
- net at C17.2, IC15.5 (BGND): now also CLKOUT3.1
- net at IC15.7 (B1_OUT): now also CLKOUT3.2
- net at C15.2, IC14.5 (BGND): now also CLKOUT2.1
- net at C15.1, IC14.6 (B2_IN), IC14.8 (BVDD): now also CLKOUT2.3
- net at IC14.7 (B1_OUT): now also CLKOUT2.2
- net at C13.1, IC13.6 (B2_IN), IC13.8 (BVDD): now also CLKOUT1.3
- net at C13.2, IC13.5 (BGND): now also CLKOUT1.1
- net at C19.1, IC16.6 (B2_IN), IC16.8 (BVDD): now also CLKOUT4.3
- net at C19.2, IC16.5 (BGND): now also CLKOUT4.1
- net at IC16.7 (B1_OUT): now also CLKOUT4.2
- net at IC13.7 (B1_OUT): now also CLKOUT1.2
