File: Hardware/harp timestamp generator Gen3/core.kicad_sch (KiCad schematic)
At the start: 21 parts, among them IC18 SN74LVC1G125DBVT, IC19 SN74LVC1G125DBVT, IC6 ATXMEGA16A4U-A

Commit message: review após 1ª produção de placas teste
> harp timestamp generator Gen3
  . mudança da case de Q2
  . mudança de ligação em 'Button0'

> harp timestamp generator Gen3 front panel
  . acerto no recorte da ficha IDC e interruptor bateria
  . modificação de setup no logo 'harp'

> harp timestamp generator Gen3 rear panel
  . acerto no recorte de ficha USB
Connections:
- net GND: now also BUTTON0.1 (A); no longer BUTTON0.3 (C)
Other:
- moved on the sheet: BUTTON0
Changed lines of the file:
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@@
 	(symbol
 		(lib_id "Switch:SW_SPDT")
-		(at 33.02 104.14 180)
+		(at 33.02 104.14 0)
+		(mirror y)
 		(unit 1)
 		(body_style 1)
@@
 		(dnp no)
 		(property "Reference" "BUTTON0"
-			(at 30.48 97.282 0)
+			(at 30.48 110.998 0)
 			(show_name no)
 			(do_not_autoplace no)
@@
 		)
 		(property "Value" "CFPA"
-			(at 30.48 99.06 0)
+			(at 30.48 109.22 0)
 			(hide yes)
 			(show_name no)
